File: canfd_breakout/canfd_breakout.kicad_sch (KiCad schematic)
At the start: 15 parts, among them J1 Conn_02x02_Odd_Even, J2 Conn_01x08, J3 Conn_01x08, U1 MCP2517FD-xSL, U2 MCP2562-E-SN, Y1 40MHz

Commit message: add pdf shematic
Other:
- company: (none) -> Pi
- title: (none) -> CAN-FD breakout board
Changed lines of the file:
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@@
 (kicad_sch (version 20230121) (generator eeschema)
   (paper "A4")
+  (title_block
+    (title "CAN-FD breakout board")
+    (date "2023-11-16")
+    (rev "1.0")
+    (company "Pi")
+  )
   (junction (at 118.11 119.38) (diameter 0) (color 0 0 0 0)
   )
